File: hardware/hardware.kicad_pcb (KiCad board)
At the start: 2 copper layers, 32 x 42 mm, 70 parts, among them J1 VCC, J10 Conn_01x05_Pin, J2 GND, J3 PHASE_A, J4 PHASE_B, J5 PHASE_C, Q1 SiR158DP, Q10 SiR158DP, Q2 SiR158DP, Q3 SiR158DP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

Commit message: additional vcc / gnd
Parts:
- added J6: VBAT+, TestPoint:TestPoint_Pad_2.0x2.0mm, F.Cu at (106.7, 62.2)
- added J7: GND, TestPoint:TestPoint_Pad_2.0x2.0mm, F.Cu at (119.1, 62.2)
Routing:
- net GND: track 235.9 -> 237.3 mm
- net VBAT+: track 65.2 -> 66.3 mm
