File: hardware/hardware.kicad_pcb (KiCad board)
At the start: 2 copper layers, 32 x 43.7 mm, 50 parts, among them J1 VBAT, J2 GND, Q1 SiR158DP, Q10 SiR158DP, Q2 SiR158DP, Q3 SiR158DP, Q4 SiR158DP, Q5 SiR158DP, Q7 BC817, Q8 BC817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

Commit message: update rev3 board
Parts:
- GND, PWM: footprint TestPoint:TestPoint_Keystone_5015_Micro-Minature -> TestPoint:TestPoint_Keystone_5015_Micro_Mini
Other:
- board text added: "NoahESC rev3"
- board text removed: "NoahESC rev2"

Commit message: add rev4
Parts:
- added J5: Programming, Connector_PinHeader_1.27mm:PinHeader_1x06_P1.27mm_Vertical, F.Cu at (99.2, 67.1)
- C2, C3: value 0.1uF -> 100nF
- renumbered GND to J3, PWM to J4
Connections:
- net PWM_CL renamed MOSI
- U1 pad 16: unconnected-(U1-PB4-Pad16) -> MISO
- U1 pad 17: unconnected-(U1-PB5-Pad17) -> SCK
- U1 pad 29: unconnected-(U1-PC6/~{RESET}-Pad29) -> RESET
Routing:
- net SCK: track 0.00 -> 31.7 mm, vias 0 -> 1
- net MISO: track 0.00 -> 19.2 mm, vias 0 -> 2
- net MOSI: track 31.8 -> 48.8 mm, vias 0 -> 2
- net RESET: track 0.00 -> 14.5 mm, vias 0 -> 2
- net 5V: track 33.2 -> 42.7 mm, vias 0 -> 2
- net GND: track 32.2 -> 38.6 mm, vias 35 -> 37
Other:
- board text added: "GND 5V RES MISO MOSI SCK"
- board text added: "NoahESC rev4"
- board text removed: "NoahESC rev3"

Commit message: add new pwm pin
Parts:
- removed J3: GND, TestPoint:TestPoint_Keystone_5015_Micro_Mini
- removed J4: PWM, TestPoint:TestPoint_Keystone_5015_Micro_Mini
- added J6: PWM, Connector_PinHeader_2.54mm:PinHeader_1x02_P2.54mm_Vertical, F.Cu at (102.4, 62.5)
Routing:
- net GND: track 38.6 -> 34.9 mm, vias 37 -> 36
Other:
- board text added: "GND PWM"
- board text added: "GND VCC"
